File: design/BLDC_4.kicad_sch (KiCad schematic)
At the start: 27 parts, among them J1 BM10B-GHS-TBT_LF__SN__N_, J2 USB_C_Receptacle, K1 SERVO, P1 CANBUS, P2 HALL/Encoder, P3 PWR_COMM, P4 IN+, P5 IN-, P6 MOTOR3, P7 MOTOR2, P8 MOTOR1

Commit message: added documentation
Parts:
- C1: The code for order (none) -> C1206C104K5RAC7210; Значение (none) -> 100 нФ; Наименование (none) -> Конденсатор керамический 100 нФ 0603; Обозначение (none) -> C; Позиционное обозначение (none) -> C1
- C2: The code for order (none) -> C1206C104K5RAC7210; Значение (none) -> 100 нФ; Наименование (none) -> Конденсатор керамический 100 нФ 0603; Обозначение (none) -> C; Позиционное обозначение (none) -> C2
- D1: The code for order (none) -> LTST-C190KRKT; Значение (none) -> RED; Наименование (none) -> Светодиод красный 0603; Обозначение (none) -> HL; Позиционное обозначение (none) -> D1
- D2: The code for order (none) -> KPG-1608CGKC-T; Значение (none) -> GREEN; Наименование (none) -> Светодиод зелёный 0603; Обозначение (none) -> HL; Позиционное обозначение (none) -> D2
- D3: The code for order (none) -> LTST-C191TGKT; Значение (none) -> LED; Наименование (none) -> Светодиод жёлтый 0603; Обозначение (none) -> HL; Позиционное обозначение (none) -> D3
- D7: The code for order (none) -> SS24; Значение (none) -> SS24; Наименование (none) -> Диод Шоттки SS24 SMA; Обозначение (none) -> VD; Позиционное обозначение (none) -> D7
- J1: The code for order (none) -> BM10B-GHS-TBT(LF)(SN)(N); Значение (none) -> BM10B-GHS-TBT; Наименование (none) -> Разъём ST BM10B-GHS-TBT 10-pin; Обозначение (none) -> XS; Позиционное обозначение (none) -> J1
- J2: The code for order (none) -> USB4205-GF-A; Значение (none) -> USB-C; Наименование (none) -> Разъём USB Type-C; Обозначение (none) -> XS; Позиционное обозначение (none) -> J2
- K1: The code for order (none) -> Servo Driver HAT (B); Значение (none) -> SERVO; Наименование (none) -> Разъём сервопривода 3-pin; Обозначение (none) -> XS; Позиционное обозначение (none) -> K1
- P1: The code for order (none) -> B4B-PH-K(LF)(SN); Значение (none) -> CANBUS; Наименование (none) -> Разъём B4B-PH-K(LF)(SN); Обозначение (none) -> XS; Позиционное обозначение (none) -> P1
- P2: The code for order (none) -> JST SM06B-SRSS-TB; Значение (none) -> HALL/Encoder; Наименование (none) -> Разъём датчика угла JST-6; Обозначение (none) -> XS; Позиционное обозначение (none) -> P2
- P3: The code for order (none) -> S7B-PH-SM4-TB; Значение (none) -> PWR_COMM; Наименование (none) -> Клеммник питания B7B-PH-KL; Обозначение (none) -> XT; Позиционное обозначение (none) -> P3
- P4: The code for order (none) -> KEYS5011; Значение (none) -> IN+; Наименование (none) -> Клеммник входа "+"; Обозначение (none) -> XT; Позиционное обозначение (none) -> P4
- P5: The code for order (none) -> KEYS5011; Значение (none) -> IN-; Наименование (none) -> Клеммник входа "-"; Обозначение (none) -> XT; Позиционное обозначение (none) -> P5
- P6: The code for order (none) -> Keystone 5015; Значение (none) -> MOTOR3; Наименование (none) -> Клеммник подключения двигателя 3; Обозначение (none) -> XT; Позиционное обозначение (none) -> P6
- P7: The code for order (none) -> Keystone 5015; Значение (none) -> MOTOR2; Наименование (none) -> Клеммник подключения двигателя 2; Обозначение (none) -> XT; Позиционное обозначение (none) -> P7
- P8: The code for order (none) -> Keystone 5015; Значение (none) -> MOTOR1; Наименование (none) -> Клеммник подключения двигателя 1; Обозначение (none) -> XT; Позиционное обозначение (none) -> P8
- R1: The code for order (none) -> 39k 0603 5%; Значение (none) -> 39 кОм; Наименование (none) -> Чип резистор 39 кОм 0603 5%; Обозначение (none) -> R; Позиционное обозначение (none) -> R1
- R10: The code for order (none) -> WSLP27262L000FEA; Значение (none) -> 0R (шунт); Наименование (none) -> Резистор-шунт 0 Ом 2 Вт; Обозначение (none) -> R; Позиционное обозначение (none) -> R10
- R103: The code for order (none) -> RC0603FR-075K11L; Значение (none) -> 5.1 кОм; Наименование (none) -> Чип резистор 5.1 кОм 0603; Обозначение (none) -> R; Позиционное обозначение (none) -> R103
- R104: The code for order (none) -> RC0603FR-075K11L; Значение (none) -> 5.1 кОм; Наименование (none) -> Чип резистор 5.1 кОм 0603; Обозначение (none) -> R; Позиционное обозначение (none) -> R104
- R11: The code for order (none) -> WSLP27262L000FEA; Значение (none) -> 0R (шунт); Наименование (none) -> Резистор-шунт 0 Ом 2 Вт; Обозначение (none) -> R; Позиционное обозначение (none) -> R11
- R2: The code for order (none) -> CR-03JL7---2K2; Значение (none) -> 2.2 кОм; Наименование (none) -> Чип резистор 2.2 кОм 0603 1%; Обозначение (none) -> R; Позиционное обозначение (none) -> R2
- R6: The code for order (none) -> 100R 1% 0603; Значение (none) -> 100 Ом; Наименование (none) -> Чип резистор 100 Ом 0603 1%; Обозначение (none) -> R; Позиционное обозначение (none) -> R6
- R7: The code for order (none) -> 100R 1% 0603; Значение (none) -> 100 Ом; Наименование (none) -> Чип резистор 100 Ом 0603 1%; Обозначение (none) -> R; Позиционное обозначение (none) -> R7
- R8: The code for order (none) -> CR-03JL7---2K2; Значение (none) -> 2.2 кОм; Наименование (none) -> Чип резистор 2.2 кОм 0603 1%; Обозначение (none) -> R; Позиционное обозначение (none) -> R8
- R9: The code for order (none) -> CR-03JL7---2K2; Значение (none) -> 2.2 кОм; Наименование (none) -> Чип резистор 2.2 кОм 0603 1%; Обозначение (none) -> R; Позиционное обозначение (none) -> R9
