File: design/CAN.kicad_sch (KiCad schematic)
At the start: 4 parts, among them U1 SN65HVD232

Commit message: added documentation
Parts:
- C3: The code for order (none) -> CL10B225KP8NNNC; Значение (none) -> 2.2 мкФ; Наименование (none) -> Конденсатор керамический 2.2 мкФ 0603; Обозначение (none) -> C; Позиционное обозначение (none) -> C3
- R12: The code for order (none) -> RC0603FR-070RL; Значение (none) -> 0R (перемычка); Наименование (none) -> Резистор-перемычка 0 Ом 0603; Обозначение (none) -> R; Позиционное обозначение (none) -> R12
- R13: The code for order (none) -> CR-03JL7---10K; Значение (none) -> 10 кОм; Наименование (none) -> Чип резистор 10 кОм 0603 1%; Обозначение (none) -> R; Позиционное обозначение (none) -> R13
- U1: The code for order (none) -> SN65HVD232DR; Значение (none) -> SN65HVD232; Наименование (none) -> CAN приёмопередатчик SN65HVD232DR; Обозначение (none) -> DA; Позиционное обозначение (none) -> U1
