File: design/Power.kicad_sch (KiCad schematic)
At the start: 48 parts, among them U3 DRV8302, U4 TC2117

Commit message: added documentation
Parts:
- C21: The code for order (none) -> CL10B225KP8NNNC; Значение (none) -> 2.2 мкФ; Наименование (none) -> Конденсатор керамический 2.2 мкФ 0603; Обозначение (none) -> C; Позиционное обозначение (none) -> C21
- C22: The code for order (none) -> CL10B225KP8NNNC; Значение (none) -> 2.2 мкФ; Наименование (none) -> Конденсатор керамический 2.2 мкФ 0603; Обозначение (none) -> C; Позиционное обозначение (none) -> C22
- C23: The code for order (none) -> CC0603JRNPO9BN121; Значение (none) -> 120 пФ; Наименование (none) -> Конденсатор керамический 120 пФ 0603; Обозначение (none) -> C; Позиционное обозначение (none) -> C23
- C24: The code for order (none) -> CL10B225KP8NNNC; Значение (none) -> 2.2 мкФ; Наименование (none) -> Конденсатор керамический 2.2 мкФ 0603; Обозначение (none) -> C; Позиционное обозначение (none) -> C24
- C25: The code for order (none) -> CL10B225KP8NNNC; Значение (none) -> 2.2 мкФ; Наименование (none) -> Конденсатор керамический 2.2 мкФ 0603; Обозначение (none) -> C; Позиционное обозначение (none) -> C25
- C26: The code for order (none) -> CL10B682KBNC; Значение (none) -> 6.8 нФ; Наименование (none) -> Конденсатор керамический 6.8 нФ 0603; Обозначение (none) -> C; Позиционное обозначение (none) -> C26
- C27: The code for order (none) -> C0603X223K101T; Значение (none) -> 22 нФ; Наименование (none) -> Конденсатор керамический 22 нФ 0603; Обозначение (none) -> C; Позиционное обозначение (none) -> C27
- C28: The code for order (none) -> CL10B225KP8NNNC; Значение (none) -> 2.2 мкФ; Наименование (none) -> Конденсатор керамический 2.2 мкФ 0603; Обозначение (none) -> C; Позиционное обозначение (none) -> C28
- C29: The code for order (none) -> 1206B105K500CT; Значение (none) -> 10 мкФ 50В; Наименование (none) -> Конденсатор керамический 10 мкФ 50В 1206; Обозначение (none) -> C; Позиционное обозначение (none) -> C29
- C30: The code for order (none) -> 1206B105K500CT; Значение (none) -> 10 мкФ 50В; Наименование (none) -> Конденсатор керамический 10 мкФ 50В 1206; Обозначение (none) -> C; Позиционное обозначение (none) -> C30
- C31: The code for order (none) -> 1206B105K500CT; Значение (none) -> 10 мкФ 50В; Наименование (none) -> Конденсатор керамический 10 мкФ 50В 1206; Обозначение (none) -> C; Позиционное обозначение (none) -> C31
- C32: The code for order (none) -> C1206C104K5RAC7210; Значение (none) -> 100 нФ; Наименование (none) -> Конденсатор керамический 100 нФ 0603; Обозначение (none) -> C; Позиционное обозначение (none) -> C32
- C33: The code for order (none) -> TCC0603X7R224K500CT; Значение (none) -> 220 нФ; Наименование (none) -> Конденсатор крамический 220 нФ X7R 0603; Обозначение (none) -> C; Позиционное обозначение (none) -> C33
- C34: The code for order (none) -> TCC0603X7R224K500CT; Значение (none) -> 220 нФ; Наименование (none) -> Конденсатор крамический 220 нФ X7R 0603; Обозначение (none) -> C; Позиционное обозначение (none) -> C34
- C35: The code for order (none) -> TCC0603X7R224K500CT; Значение (none) -> 220 нФ; Наименование (none) -> Конденсатор крамический 220 нФ X7R 0603; Обозначение (none) -> C; Позиционное обозначение (none) -> C35
- C36: The code for order (none) -> CL10B222KB8NNNC; Значение (none) -> 2.2 нФ; Наименование (none) -> Конденсатор керамический 2.2 нФ 0603; Обозначение (none) -> C; Позиционное обозначение (none) -> C36
- C37: The code for order (none) -> CL10B222KB8NNNC; Значение (none) -> 2.2 нФ; Наименование (none) -> Конденсатор керамический 2.2 нФ 0603; Обозначение (none) -> C; Позиционное обозначение (none) -> C37
- C38: The code for order (none) -> CL10B225KP8NNNC; Значение (none) -> 2.2 мкФ; Наименование (none) -> Конденсатор керамический 2.2 мкФ 0603; Обозначение (none) -> C; Позиционное обозначение (none) -> C38
- C39: The code for order (none) -> T491D107K010AT; Значение (none) -> 100 мкФ; Наименование (none) -> Конденсатор танталовый 100 мкФ 10В; Обозначение (none) -> C; Позиционное обозначение (none) -> C39
- C40: The code for order (none) -> 1206B105K500CT; Значение (none) -> 10 мкФ 50В; Наименование (none) -> Конденсатор керамический 10 мкФ 50В 1206; Обозначение (none) -> C; Позиционное обозначение (none) -> C40
- C41: The code for order (none) -> T491D107K010AT; Значение (none) -> 100 мкФ; Наименование (none) -> Конденсатор танталовый 100 мкФ 10В; Обозначение (none) -> C; Позиционное обозначение (none) -> C41
- C42: The code for order (none) -> 1206B105K500CT; Значение (none) -> 10 мкФ 50В; Наименование (none) -> Конденсатор керамический 10 мкФ 50В 1206; Обозначение (none) -> C; Позиционное обозначение (none) -> C42
- C43: The code for order (none) -> 1206B105K500CT; Значение (none) -> 10 мкФ 50В; Наименование (none) -> Конденсатор керамический 10 мкФ 50В 1206; Обозначение (none) -> C; Позиционное обозначение (none) -> C43
- C44: The code for order (none) -> C5750X7R2A155K230KA; Значение (none) -> 15 мкФ 100В; Наименование (none) -> Конденсатор керамический 15 мкФ 100В 2220; Обозначение (none) -> C; Позиционное обозначение (none) -> C44
- C45: The code for order (none) -> 1206B105K500CT; Значение (none) -> 10 мкФ 50В; Наименование (none) -> Конденсатор керамический 10 мкФ 50В 1206; Обозначение (none) -> C; Позиционное обозначение (none) -> C45
- C46: The code for order (none) -> 1206B105K500CT; Значение (none) -> 10 мкФ 50В; Наименование (none) -> Конденсатор керамический 10 мкФ 50В 1206; Обозначение (none) -> C; Позиционное обозначение (none) -> C46
- C47: value 15u,100V -> 15u,100v; The code for order (none) -> C5750X7R2A155K230KA; Значение (none) -> 15 мкФ 100В; Наименование (none) -> Конденсатор керамический 15 мкФ 100В 2220; Обозначение (none) -> C; Позиционное обозначение (none) -> C47
- D4: The code for order (none) -> 1N5819; Значение (none) -> 1N5819; Наименование (none) -> Диод Шоттки 1N5819; Обозначение (none) -> VD; Позиционное обозначение (none) -> D4
- D5: The code for order (none) -> SMAJ5.0A; Значение (none) -> SMAJ5.0A; Наименование (none) -> Защитный диод SMAJ7.0A; Обозначение (none) -> VD; Позиционное обозначение (none) -> D5
- L1: The code for order (none) -> B82422H1223K000; Значение (none) -> 22 мкГн; Наименование (none) -> Дроссель 22 мкГн 8x5 мм; Обозначение (none) -> L; Позиционное обозначение (none) -> L1
- R23: The code for order (none) -> 18k 1% 0603; Значение (none) -> 18 кОм; Наименование (none) -> Чип резистор 18 кОм 0603 1%; Обозначение (none) -> R; Позиционное обозначение (none) -> R23
- R24: The code for order (none) -> CR-03JL7---3K3; Значение (none) -> 3.3 кОм; Наименование (none) -> Чип резистор 3.3 кОм 0603 1%; Обозначение (none) -> R; Позиционное обозначение (none) -> R24
- R25: The code for order (none) -> CR-03JL7---10K; Значение (none) -> 10 кОм; Наименование (none) -> Чип резистор 10 кОм 0603 1%; Обозначение (none) -> R; Позиционное обозначение (none) -> R25
- R26: The code for order (none) -> 15k 0603 5%; Значение (none) -> 15 кОм; Наименование (none) -> Чип резистор 15 кОм 0603 5%; Обозначение (none) -> R; Позиционное обозначение (none) -> R26
- R27: The code for order (none) -> 220k 0603 5%; Значение (none) -> 220 кОм; Наименование (none) -> Чип резистор 220 кОм 0603 5%; Обозначение (none) -> R; Позиционное обозначение (none) -> R27
- R28: The code for order (none) -> 1M 1% 0603; Значение (none) -> 1 МОм; Наименование (none) -> Чип резистор 1 МОм 0603 1%; Обозначение (none) -> R; Позиционное обозначение (none) -> R28
- R29: The code for order (none) -> 100R 1% 0603; Значение (none) -> 100 Ом; Наименование (none) -> Чип резистор 100 Ом 0603 1%; Обозначение (none) -> R; Позиционное обозначение (none) -> R29
- R30: The code for order (none) -> 100R 1% 0603; Значение (none) -> 100 Ом; Наименование (none) -> Чип резистор 100 Ом 0603 1%; Обозначение (none) -> R; Позиционное обозначение (none) -> R30
- R31: The code for order (none) -> 100R 1% 0603; Значение (none) -> 100 Ом; Наименование (none) -> Чип резистор 100 Ом 0603 1%; Обозначение (none) -> R; Позиционное обозначение (none) -> R31
- R32: The code for order (none) -> 100R 1% 0603; Значение (none) -> 100 Ом; Наименование (none) -> Чип резистор 100 Ом 0603 1%; Обозначение (none) -> R; Позиционное обозначение (none) -> R32
- R33: The code for order (none) -> 39k 0603 5%; Значение (none) -> 39 кОм; Наименование (none) -> Чип резистор 39 кОм 0603 5%; Обозначение (none) -> R; Позиционное обозначение (none) -> R33
- R34: The code for order (none) -> CR-03JL7---2K2; Значение (none) -> 2.2 кОм; Наименование (none) -> Чип резистор 2.2 кОм 0603 1%; Обозначение (none) -> R; Позиционное обозначение (none) -> R34
- R35: The code for order (none) -> 39k 0603 5%; Значение (none) -> 39 кОм; Наименование (none) -> Чип резистор 39 кОм 0603 5%; Обозначение (none) -> R; Позиционное обозначение (none) -> R35
- R36: The code for order (none) -> CR-03JL7---2K2; Значение (none) -> 2.2 кОм; Наименование (none) -> Чип резистор 2.2 кОм 0603 1%; Обозначение (none) -> R; Позиционное обозначение (none) -> R36
- R37: The code for order (none) -> 39k 0603 5%; Значение (none) -> 39 кОм; Наименование (none) -> Чип резистор 39 кОм 0603 5%; Обозначение (none) -> R; Позиционное обозначение (none) -> R37
- R38: The code for order (none) -> CR-03JL7---2K2; Значение (none) -> 2.2 кОм; Наименование (none) -> Чип резистор 2.2 кОм 0603 1%; Обозначение (none) -> R; Позиционное обозначение (none) -> R38
- U3: The code for order (none) -> DRV8302DCA; Значение (none) -> DRV8302; Наименование (none) -> Драйвер двигателя DRV8302DCA; Обозначение (none) -> DA; Позиционное обозначение (none) -> U3
- U4: The code for order (none) -> BCP51; Значение (none) -> TC2117; Наименование (none) -> Стабилизатор напряжения TC2117; Обозначение (none) -> DA; Позиционное обозначение (none) -> U4
