File: design/hall_filters.kicad_sch (KiCad schematic)
At the start: 11 parts

Commit message: added documentation
Parts:
- C4: The code for order (none) -> MSCC0603-4N7J; Значение (none) -> 4.7 нФ; Наименование (none) -> Конденсатор керамический 4.7 нФ 0603; Обозначение (none) -> C; Позиционное обозначение (none) -> C4
- C5: The code for order (none) -> MSCC0603-4N7J; Значение (none) -> 4.7 нФ; Наименование (none) -> Конденсатор керамический 4.7 нФ 0603; Обозначение (none) -> C; Позиционное обозначение (none) -> C5
- C6: The code for order (none) -> MSCC0603-4N7J; Значение (none) -> 4.7 нФ; Наименование (none) -> Конденсатор керамический 4.7 нФ 0603; Обозначение (none) -> C; Позиционное обозначение (none) -> C6
- C7: The code for order (none) -> MSCC0603-4N7J; Значение (none) -> 4.7 нФ; Наименование (none) -> Конденсатор керамический 4.7 нФ 0603; Обозначение (none) -> C; Позиционное обозначение (none) -> C7
- R14: The code for order (none) -> CR-03JL7---10K; Значение (none) -> 10 кОм; Наименование (none) -> Чип резистор 10 кОм 0603 1%; Обозначение (none) -> R; Позиционное обозначение (none) -> R14
- R15: The code for order (none) -> CR-03JL7---2K2; Значение (none) -> 2.2 кОм; Наименование (none) -> Чип резистор 2.2 кОм 0603 1%; Обозначение (none) -> R; Позиционное обозначение (none) -> R15
- R16: The code for order (none) -> CR-03JL7---2K2; Значение (none) -> 2.2 кОм; Наименование (none) -> Чип резистор 2.2 кОм 0603 1%; Обозначение (none) -> R; Позиционное обозначение (none) -> R16
- R17: The code for order (none) -> CR-03JL7---2K2; Значение (none) -> 2.2 кОм; Наименование (none) -> Чип резистор 2.2 кОм 0603 1%; Обозначение (none) -> R; Позиционное обозначение (none) -> R17
- R18: The code for order (none) -> CR-03JL7---10K; Значение (none) -> 10 кОм; Наименование (none) -> Чип резистор 10 кОм 0603 1%; Обозначение (none) -> R; Позиционное обозначение (none) -> R18
- R19: The code for order (none) -> CR-03JL7---10K; Значение (none) -> 10 кОм; Наименование (none) -> Чип резистор 10 кОм 0603 1%; Обозначение (none) -> R; Позиционное обозначение (none) -> R19
- R20: The code for order (none) -> CR-03JL7---10K; Значение (none) -> 10 кОм; Наименование (none) -> Чип резистор 10 кОм 0603 1%; Обозначение (none) -> R; Позиционное обозначение (none) -> R20
