File: design/mosfets.kicad_sch (KiCad schematic)
At the start: 15 parts, among them Q1 IRFS7530, Q2 IRFS7530, Q3 IRFS7530, Q4 IRFS7530, Q5 IRFS7530, Q6 IRFS7530

Commit message: added documentation
Parts:
- Q1: The code for order (none) -> IRFS7530TRLPBF; Значение (none) -> IRFS7530; Наименование (none) -> Транзистор IRFS7530TRLPBF; Обозначение (none) -> VT; Позиционное обозначение (none) -> Q1
- Q2: The code for order (none) -> IRFS7530TRLPBF; Значение (none) -> IRFS7530; Наименование (none) -> Транзистор IRFS7530TRLPBF; Обозначение (none) -> VT; Позиционное обозначение (none) -> Q2
- Q3: The code for order (none) -> IRFS7530TRLPBF; Значение (none) -> IRFS7530; Наименование (none) -> Транзистор IRFS7530TRLPBF; Обозначение (none) -> VT; Позиционное обозначение (none) -> Q3
- Q4: The code for order (none) -> IRFS7530TRLPBF; Значение (none) -> IRFS7530; Наименование (none) -> Транзистор IRFS7530TRLPBF; Обозначение (none) -> VT; Позиционное обозначение (none) -> Q4
- Q5: The code for order (none) -> IRFS7530TRLPBF; Значение (none) -> IRFS7530; Наименование (none) -> Транзистор IRFS7530TRLPBF; Обозначение (none) -> VT; Позиционное обозначение (none) -> Q5
- Q6: The code for order (none) -> IRFS7530TRLPBF; Значение (none) -> IRFS7530; Наименование (none) -> Транзистор IRFS7530TRLPBF; Обозначение (none) -> VT; Позиционное обозначение (none) -> Q6
- R39: The code for order (none) -> CR-03JL7---4R7; Значение (none) -> 4.7 Ом; Наименование (none) -> Чип резистор 4.7 Ом 0603 1%; Обозначение (none) -> R; Позиционное обозначение (none) -> R39
- R40: The code for order (none) -> CR-03JL7---4R7; Значение (none) -> 4.7 Ом; Наименование (none) -> Чип резистор 4.7 Ом 0603 1%; Обозначение (none) -> R; Позиционное обозначение (none) -> R40
- R41: The code for order (none) -> 39k 0603 5%; Значение (none) -> 39 кОм; Наименование (none) -> Чип резистор 39 кОм 0603 5%; Обозначение (none) -> R; Позиционное обозначение (none) -> R41
- R42: The code for order (none) -> CR-03JL7---4R7; Значение (none) -> 4.7 Ом; Наименование (none) -> Чип резистор 4.7 Ом 0603 1%; Обозначение (none) -> R; Позиционное обозначение (none) -> R42
- R43: The code for order (none) -> CR-03JL7---4R7; Значение (none) -> 4.7 Ом; Наименование (none) -> Чип резистор 4.7 Ом 0603 1%; Обозначение (none) -> R; Позиционное обозначение (none) -> R43
- R44: The code for order (none) -> 39k 0603 5%; Значение (none) -> 39 кОм; Наименование (none) -> Чип резистор 39 кОм 0603 5%; Обозначение (none) -> R; Позиционное обозначение (none) -> R44
- R45: The code for order (none) -> CR-03JL7---4R7; Значение (none) -> 4.7 Ом; Наименование (none) -> Чип резистор 4.7 Ом 0603 1%; Обозначение (none) -> R; Позиционное обозначение (none) -> R45
- R46: The code for order (none) -> CR-03JL7---4R7; Значение (none) -> 4.7 Ом; Наименование (none) -> Чип резистор 4.7 Ом 0603 1%; Обозначение (none) -> R; Позиционное обозначение (none) -> R46
- R47: The code for order (none) -> 39k 0603 5%; Значение (none) -> 39 кОм; Наименование (none) -> Чип резистор 39 кОм 0603 5%; Обозначение (none) -> R; Позиционное обозначение (none) -> R47
