File: design/temp.kicad_sch (KiCad schematic)
At the start: 3 parts

Commit message: added documentation
Parts:
- C8: The code for order (none) -> CL10B225KP8NNNC; Значение (none) -> 2.2 мкФ; Наименование (none) -> Конденсатор керамический 2.2 мкФ 0603; Обозначение (none) -> C; Позиционное обозначение (none) -> C8
- R21: The code for order (none) -> CR-03JL7---10K; Значение (none) -> NTC 10кОм; Наименование (none) -> Термистор NTC 10 кОм 0603; Обозначение (none) -> RK; Позиционное обозначение (none) -> R21
- R22: The code for order (none) -> CR-03JL7---10K; Значение (none) -> 10 кОм; Наименование (none) -> Чип резистор 10 кОм 0603 1%; Обозначение (none) -> R; Позиционное обозначение (none) -> R22
Changed lines of the file:
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@@
+			)
+		)
+		(property "The code for order" "CR-03JL7---10K"
+			(at 111.76 86.36 0)
+			(effects
+				(font
+					(size 1.27 1.27)
+				)
+				(hide yes)
+			)
+		)
+		(property "Значение" "NTC 10кОм"
+			(at 111.76 86.36 0)
+			(effects
+				(font
+					(size 1.27 1.27)
+				)
+				(hide yes)
+			)
+		)
+		(property "Наименование" "Термистор NTC 10 кОм 0603"
+			(at 111.76 86.36 0)
+			(effects
+				(font
+					(size 1.27 1.27)
+				)
+				(hide yes)
+			)
+		)
+		(property "Обозначение" "RK"
+			(at 111.76 86.36 0)
+			(effects
+				(font
+					(size 1.27 1.27)
+				)
+				(hide yes)
+			)
+		)
+		(property "Позиционное обозначение" "R21"
+			(at 111.76 86.36 0)
+			(effects
+				(font
+					(size 1.27 1.27)
+				)
+				(hide yes)
 			)
 		)
@@
 			)
 		)
+		(property "The code for order" "CR-03JL7---10K"
+			(at 111.76 104.14 0)
+			(effects
+				(font
+					(size 1.27 1.27)
+				)
+				(hide yes)
+			)
+		)
+		(property "Значение" "10 кОм"
+			(at 111.76 104.14 0)
+			(effects
+				(font
+					(size 1.27 1.27)
+				)
+				(hide yes)
+			)
+		)
+		(property "Наименование" "Чип резистор 10 кОм 0603 1%"
+			(at 111.76 104.14 0)
+			(effects
+				(font
+					(size 1.27 1.27)
+				)
+				(hide yes)
+			)
+		)
+		(property "Обозначение" "R"
+			(at 111.76 104.14 0)
+			(effects
+				(font
+					(size 1.27 1.27)
+				)
+				(hide yes)
+			)
+		)
+		(property "Позиционное обозначение" "R22"
+			(at 111.76 104.14 0)
+			(effects
+				(font
+					(size 1.27 1.27)
+				)
+				(hide yes)
+			)
+		)
 		(pin "1"
 		)
@@
 			)
 		)
+		(property "The code for order" "CL10B225KP8NNNC"
+			(at 105.41 104.14 0)
+			(effects
+				(font
+					(size 1.27 1.27)
+				)
+				(hide yes)
+			)
+		)
+		(property "Значение" "2.2 мкФ"
+			(at 105.41 104.14 0)
+			(effects
+				(font
+					(size 1.27 1.27)
+				)
+				(hide yes)
+			)
+		)
+		(property "Наименование" "Конденсатор керамический 2.2 мкФ 0603"
+			(at 105.41 104.14 0)
+			(effects
+				(font
+					(size 1.27 1.27)
+				)
+				(hide yes)
+			)
+		)
+		(property "Обозначение" "C"
+			(at 105.41 104.14 0)
+			(effects
+				(font
+					(size 1.27 1.27)
+				)
+				(hide yes)
+			)
+		)
+		(property "Позиционное обозначение" "C8"
+			(at 105.41 104.14 0)
+			(effects
+				(font
+					(size 1.27 1.27)
+				)
+				(hide yes)
+			)
+		)
